File: Pheripheral.kicad_sch (KiCad schematic)
At the start: 1 part

Commit message: updated aux
Parts:
- added C17: 1uf/6.3v, symbol Device:C
- added C18, C21, C71: 100nf/16v, symbol Device:C
- added C22, C25, C26: 4.7uf/6.3v, symbol Device:C
- added C23, C24: 5pf/50v NC, symbol Device:C
- added R12, R13, R38: 4.7K, symbol Device:R
- added R14: 24.3K, symbol Device:R
- added R15, R16: 10K/1% NC, symbol Device:R
- added R17: 5.1K/1%, symbol Device:R
- added R18, R19: 0, symbol Device:R
- U2: footprint (none) -> MT7628:MT7628_footprint
Connections:
- net REF_CLK0: now reaches U2.136 (REF_CLK0)
- net at U2.137 (WDT_RST_N): now also R38.2
- net PORST_N: now reaches U2.138 (PORST_N)
- net WLED_N: now reaches U2.144 (WLED_N)
- net UART_TXD1: now reaches U2.147 (UART_TXD1)
- net UART_RXD1: now reaches U2.148 (UART_RXD1)
- net I2S_DI: now reaches U2.16 (I2S_SDI)
- net I2S_D0: now reaches U2.17 (I2S_SDO)
- net I2S_WS: now reaches U2.18 (I2S_WS)
- net I2S_CLK: now reaches U2.19 (I2S_CLK)
- net I2C_SCLK: now reaches U2.20 (I2C_SCLK)
- net I2C_SCLK: now also R13.1
- net I2C_SD: now reaches U2.21 (I2C_SD)
- net I2C_SD: now also R12.1
- net SPI_CS1: now reaches U2.24 (SPI_CS1)
- net SPI_CLK: now reaches U2.25 (SPI_CLK)
- net SPI_MISO: now reaches U2.26 (SPI_MISO)
- net SPI_M0SI: now reaches U2.27 (SPI_MOSI)
- net SPI_CS0: now reaches U2.28 (SPI_CS0)
- net GPIO_0: now reaches U2.29 (GPIO0)
- net UART_TXD0: now reaches U2.30 (UART_TXD0)
- net UART_RXD0: now reaches U2.31 (UART_RXD0)
- net WIFI_RESET: now reaches U2.139 (EPHY_LED4_N_JTRST_N)
- net EPH_LED1_N: now reaches U2.142 (EPHY_LED1_N_JTDI)
- net EPH_LED0_N: now reaches U2.143 (EPHY_LED0_N_JTDO)
- net 3.3VD: now reaches U2.32 (AVDD33_TX_P0)
- net 3.3VD: now also U2.131 (AVDD12_PCIE), U2.38 (AVDD33_COM), U2.41 (AVDD33_TX_P1234_1), U2.53 (AVDD33_TX_P1234_2), U2.60 (AVDD33_USB), C17.1, C18.1, C21.1, C22.1, C26.2, C71.1, R12.2, R13.2, R38.1
- net RXIP0: now reaches U2.33 (MDI_RP_P0)
- net RXIN0: now reaches U2.34 (MDI_RN_P0)
- net TXOP0: now reaches U2.35 (MDI_TP_P0)
- net TXON0: now reaches U2.36 (MDI_TN_P0)
- net at U2.39 (EPHY_VRT): now also R14.2
- net TXOP1: now reaches U2.40 (MDI_TP_P1)
- net TXON1: now reaches U2.42 (MDI_TN_P1)
- net RXIP1: now reaches U2.43 (MDI_RP_P1)
- net RXIN1: now reaches U2.44 (MDI_RN_P1)
- net PWM_CH0: now reaches U2.45 (MDI_RP_P2)
- net PWM_CH1: now reaches U2.46 (MDI_RN_P2)
- net UART_RXD2: now reaches U2.47 (MDI_TP_P2)
- net UART_TXD2: now reaches U2.48 (MDI_TN_P2)
- net SD_WP: now reaches U2.49 (MDI_TP_P3)
- net SD_WP: now also R16.1
- net SD_CD: now reaches U2.50 (MDI_TN_P3)
- net SD_CD: now also R15.1
- net SD_D1: now reaches U2.51 (MDI_RP_P3)
- net SD_D0: now reaches U2.52 (MDI_RN_P3)
- net SD_CLK: now reaches U2.54 (MDI_RP_P4)
- net SD_CMD: now reaches U2.55 (MDI_RN_P4)
- net SD_D3: now reaches U2.56 (MDI_TP_P4)
- net SD_D2: now reaches U2.57 (MDI_TN_P4)
- net GND: now reaches U2.128 (PCIE_IO_VSS)
- net GND: now also C17.2, C18.2, C21.2, C22.2, C23.2, C24.2, C25.1, C26.1, C71.2, R14.1, R15.2, R16.2, R17.1
- net SOC_1.2VD_MT7688: now reaches U2.134 (AVDD33_PCIE)
- net SOC_1.2VD_MT7688: now also C25.2
- net PERST_N: now reaches U2.135 (PERST_N)
- net at U2.59 (USB_VRT): now also R17.2
- net at U2.61 (USB_DP): now also R18.2
- net at U2.62 (USB_DM): now also R19.2
- new net USB_D+: C23.1, R18.1
- new net USB_D-: C24.1, R19.1
- no-connect marks 0 -> 9
Other:
- moved on the sheet: U2C, U2D, U2E

Commit message: init_sch
Parts:
- R12, R13, R38: footprint (none) -> Resistor_SMD:R_0402_1005Metric; LCSC (none) -> C25900
Changed lines of the file:
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@@
 			)
 		)
-		(property "Footprint" ""
+		(property "Footprint" "Resistor_SMD:R_0402_1005Metric"
 			(at 45.72 51.308 90)
 			(effects
@@
 		(property "Description" "Resistor"
 			(at 45.72 49.53 0)
+			(effects
+				(font
+					(size 1.27 1.27)
+				)
+				(hide yes)
+			)
+		)
+		(property "LCSC" "C25900"
+			(at 45.72 49.53 90)
 			(effects
 				(font
@@
 			)
 		)
-		(property "Footprint" ""
+		(property "Footprint" "Resistor_SMD:R_0402_1005Metric"
 			(at 36.068 35.56 90)
 			(effects
@@
 		(property "Description" "Resistor"
 			(at 34.29 35.56 0)
+			(effects
+				(font
+					(size 1.27 1.27)
+				)
+				(hide yes)
+			)
+		)
+		(property "LCSC" "C25900"
+			(at 34.29 35.56 90)
 			(effects
 				(font
@@
 			)
 		)
-		(property "Footprint" ""
+		(property "Footprint" "Resistor_SMD:R_0402_1005Metric"
 			(at 41.148 34.29 90)
 			(effects
@@
 			(effects
 				(font
+					(size 1.27 1.27)
+				)
+				(hide yes)
+			)
+		)
+		(property "LCSC" "C25900"
+			(at 39.37 34.29 90)
+			(effects
+				(font

Commit message: updated
Parts:
- C17: footprint (none) -> Capacitor_SMD:C_0402_1005Metric; LCSC (none) -> C15684
- C18, C21, C71: footprint (none) -> Capacitor_SMD:C_0402_1005Metric; LCSC (none) -> C1525
- C19: renamed from C25; footprint (none) -> Capacitor_SMD:C_0603_1608Metric; LCSC (none) -> C8032
- C20: renamed from C26; footprint (none) -> Capacitor_SMD:C_0603_1608Metric; LCSC (none) -> C8032
- C22: footprint (none) -> Capacitor_SMD:C_0603_1608Metric; LCSC (none) -> C8032
- C23, C24: footprint (none) -> Capacitor_SMD:C_0402_1005Metric; LCSC (none) -> C1573
- R14: footprint (none) -> Resistor_SMD:R_0402_1005Metric; LCSC (none) -> C102920
- R15, R16: footprint (none) -> Resistor_SMD:R_0402_1005Metric; LCSC (none) -> C25744
- R17: footprint (none) -> Capacitor_SMD:C_0402_1005Metric; LCSC (none) -> C25905
- R18, R19: footprint (none) -> Resistor_SMD:R_0402_1005Metric; LCSC (none) -> C17168
Connections:
- net 3.3VD: now also C19.2, U2.134 (AVDD33_PCIE); no longer C20.2, U2.131 (AVDD12_PCIE)
- net SOC_1.2VD_MT7688: now also C20.2, U2.131 (AVDD12_PCIE); no longer C19.2, U2.134 (AVDD33_PCIE)
Changed lines of the file:
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@@
 	(wire
 		(pts
-			(xy 149.86 91.44) (xy 143.51 91.44)
+			(xy 158.75 91.44) (xy 143.51 91.44)
 		)
 		(stroke
@@
 			)
 		)
-		(property "Footprint" ""
+		(property "Footprint" "Capacitor_SMD:C_0402_1005Metric"
 			(at 127.9652 34.29 0)
 			(effects
@@
 			)
 		)
+		(property "LCSC" "C1525"
+			(at 127 30.48 0)
+			(effects
+				(font
+					(size 1.27 1.27)
+				)
+				(hide yes)
+			)
+		)
 		(pin "2"
 		)
@@
 			)
 		)
-		(property "Footprint" ""
+		(property "Footprint" "Resistor_SMD:R_0402_1005Metric"
 			(at 105.41 105.918 90)
 			(effects
@@
 			)
 		)
+		(property "LCSC" "C17168"
+			(at 105.41 104.14 90)
+			(effects
+				(font
+					(size 1.27 1.27)
+				)
+				(hide yes)
+			)
+		)
 		(pin "2"
 		)
@@
 			)
 		)
-		(property "Footprint" ""
+		(property "Footprint" "Resistor_SMD:R_0402_1005Metric"
 			(at 105.41 109.728 90)
 			(effects
@@
 			)
 		)
+		(property "LCSC" "C17168"
+			(at 105.41 107.95 90)
+			(effects
+				(font
+					(size 1.27 1.27)
+				)
+				(hide yes)
+			)
+		)
 		(pin "2"
 		)
@@
 			)
 		)
-		(property "Footprint" ""
+		(property "Footprint" "Capacitor_SMD:C_0402_1005Metric"
 			(at 87.3252 115.57 0)
 			(effects
@@
 			)
 		)
+		(property "LCSC" "C1573"
+			(at 86.36 111.76 0)
+			(effects
+				(font
+					(size 1.27 1.27)
+				)
+				(hide yes)
+			)
+		)
 		(pin "2"
 		)
@@
 			)
 		)
-		(property "Footprint" ""
+		(property "Footprint" "Capacitor_SMD:C_0402_1005Metric"
 			(at 83.5152 111.76 0)
 			(effects
@@
 			)
 		)
+		(property "LCSC" "C1573"
+			(at 82.55 107.95 0)
+			(effects
+				(font
+					(size 1.27 1.27)
+				)
+				(hide yes)
+			)
+		)
 		(pin "2"
 		)
@@
 		(on_board yes)
 		(dnp no)
-		(property "Reference" "C26"
+		(property "Reference" "C20"
 			(at 151.384 83.058 0)
 			(effects
@@
 			)
 		)
-		(property "Footprint" ""
+		(property "Footprint" "Capacitor_SMD:C_0603_1608Metric"
 			(at 152.0952 88.9 0)
 			(effects
@@
 			)
 		)
+		(property "LCSC" "C8032"
+			(at 151.13 85.09 0)
+			(effects
+				(font
+					(size 1.27 1.27)
+				)
+				(hide yes)
+			)
+		)
 		(pin "2"
 		)
@@
 			(project "mt7628v1"
 				(path "/144686d4-2b77-460c-9924-cc86faff7e9d/218ba002-e319-46e9-a80e-651bdbb44c2c"
-					(reference "C26")
+					(reference "C20")
 					(unit 1)
 				)
@@
 			)
 		)
-		(property "Footprint" ""
+		(property "Footprint" "Capacitor_SMD:C_0402_1005Metric"
 			(at 89.8652 97.79 0)
 			(effects
@@
 			)
 		)
+		(property "LCSC" "C1525"
+			(at 88.9 93.98 0)
+			(effects
+				(font
+					(size 1.27 1.27)
+				)
+				(hide yes)
+			)
+		)
 		(pin "2"
 		)
@@
 			)
 		)
-		(property "Footprint" ""
+		(property "Footprint" "Capacitor_SMD:C_0402_1005Metric"
 			(at 101.6 100.838 90)
 			(effects
@@
 			)
 		)
+		(property "LCSC" "C25905"
+			(at 101.6 99.06 90)
+			(effects
+				(font
+					(size 1.27 1.27)
+				)
+				(hide yes)
+			)
+		)
 		(pin "2"
 		)
@@
 			)
 		)
-		(property "Footprint" ""
+		(property "Footprint" "Capacitor_SMD:C_0402_1005Metric"
 			(at 138.1252 34.29 0)
 			(effects
@@
 			)
 		)
+		(property "LCSC" "C1525"
+			(at 137.16 30.48 0)
+			(effects
+				(font
+					(size 1.27 1.27)
+				)
+				(hide yes)
+			)
+		)
 		(pin "2"
 		)
@@
 			)
 		)
-		(property "Footprint" ""
+		(property "Footprint" "Resistor_SMD:R_0402_1005Metric"
 			(at 199.39 41.148 90)
 			(effects
@@
 			)
 		)
+		(property "LCSC" "C25744"
+			(at 199.39 39.37 90)
+			(effects
+				(font
+					(size 1.27 1.27)
+				)
+				(hide yes)
+			)
+		)
 		(pin "2"
 		)
@@
 			)
 		)
-		(property "Footprint" ""
+		(property "Footprint" "Resistor_SMD:R_0402_1005Metric"
 			(at 144.78 39.878 90)
 			(effects
@@
 			)
 		)
+		(property "LCSC" "C102920"
+			(at 144.78 38.1 90)
+			(effects
+				(font
+					(size 1.27 1.27)
+				)
+				(hide yes)
+			)
+		)
 		(pin "2"
 		)
@@
 	(symbol
 		(lib_id "MT7688AN_Power-altium-import:3.3VD_CIRCLE")
-		(at 149.86 91.44 90)
+		(at 162.56 88.9 90)
 		(unit 1)
 		(exclude_from_sim no)
@@
 		(dnp no)
 		(property "Reference" "#PWR031"
-			(at 149.86 91.44 0)
+			(at 162.56 88.9 0)
 			(effects
 				(font
@@
 		)
 		(property "Value" "SOC_1.2VD_MT7688"
-			(at 153.924 92.964 90)
+			(at 168.656 86.868 90)
 			(effects
 				(font
@@
 		)
 		(property "Footprint" ""
-			(at 149.86 91.44 0)
+			(at 162.56 88.9 0)
 			(effects
 				(font
@@
 		)
 		(property "Datasheet" ""
-			(at 149.86 91.44 0)
+			(at 162.56 88.9 0)
 			(effects
 				(font
@@
 		)
 		(property "Description" ""
-			(at 149.86 91.44 0)
+			(at 162.56 88.9 0)
 			(effects
 				(font
@@
 			)
 		)
-		(property "Footprint" ""
+		(property "Footprint" "Capacitor_SMD:C_0402_1005Metric"
 			(at 116.5352 34.29 0)
 			(effects
@@
 			)
 		)
+		(property "LCSC" "C15684"
+			(at 115.57 30.48 0)
+			(effects
+				(font
+					(size 1.27 1.27)
+				)
+				(hide yes)
+			)
+		)
 		(pin "2"
 		)
@@
 			)
 		)
-		(property "Footprint" ""
+		(property "Footprint" "Resistor_SMD:R_0402_1005Metric"
 			(at 199.39 36.068 90)
 			(effects
@@
 			)
 		)
+		(property "LCSC" "C25744"
+			(at 199.39 34.29 90)
+			(effects
+				(font
+					(size 1.27 1.27)
+				)
+				(hide yes)
+			)
+		)
 		(pin "2"
 		)
@@
 		(on_board yes)
 		(dnp no)
-		(property "Reference" "C25"
+		(property "Reference" "C19"
 			(at 143.764 85.598 0)
 			(effects
@@
 			)
 		)
-		(property "Footprint" ""
+		(property "Footprint" "Capacitor_SMD:C_0603_1608Metric"
 			(at 144.4752 91.44 0)
 			(effects
@@
 			)
 		)
+		(property "LCSC" "C8032"
+			(at 143.51 87.63 0)
+			(effects
+				(font
+					(size 1.27 1.27)
+				)
+				(hide yes)
+			)
+		)
 		(pin "2"
 		)
@@
 			(project "mt7628v1"
 				(path "/144686d4-2b77-460c-9924-cc86faff7e9d/218ba002-e319-46e9-a80e-651bdbb44c2c"
-					(reference "C25")
+					(reference "C19")
 					(unit 1)
 				)
@@
 	(symbol
 		(lib_id "MT7688AN_Power-altium-import:3.3VD_CIRCLE")
-		(at 162.56 88.9 90)
+		(at 158.75 91.44 90)
 		(unit 1)
 		(exclude_from_sim no)
@@
 		(dnp no)
 		(property "Reference" "#PWR032"
-			(at 162.56 88.9 0)
+			(at 158.75 91.44 0)
 			(effects
 				(font
@@
 		)
 		(property "Value" "3.3VD"
-			(at 164.338 87.376 90)
+			(at 160.528 89.916 90)
 			(effects
 				(font
@@
 		)
 		(property "Footprint" ""
-			(at 162.56 88.9 0)
+			(at 158.75 91.44 0)
 			(effects
 				(font
@@
 		)
 		(property "Datasheet" ""
-			(at 162.56 88.9 0)
+			(at 158.75 91.44 0)
 			(effects
 				(font
@@
 		)
 		(property "Description" ""
-			(at 162.56 88.9 0)
+			(at 158.75 91.44 0)
 			(effects
 				(font
@@
 			)
 		)
-		(property "Footprint" ""
+		(property "Footprint" "Capacitor_SMD:C_0603_1608Metric"
 			(at 78.4352 97.79 0)
 			(effects
@@
 			(at 77.47 93.98 0)
 			(effects
+				(font
+					(size 1.27 1.27)
+				)
+				(hide yes)
+			)
+		)
+		(property "LCSC" "C8032"
+			(at 77.47 93.98 0)
+			(effects

Commit message: f_ver
Parts:
- added R11: 22, Resistor_SMD:R_0402_1005Metric, symbol MT7688AN_Reset-altium-import:root_2_Res1_Miscellaneous Devices.SchLib
- U2: footprint MT7628:MT7628_footprint -> Library:MT7628_footprint
Connections:
- net SPI_CLK: now also R11.1; no longer U2.25 (SPI_CLK)
- net SPI_M0SI renamed SPI_MOSI
- new net: R11.2, U2.25 (SPI_CLK)
Changed lines of the file:
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@@
 	(wire
 		(pts
+			(xy 43.18 29.21) (xy 43.18 30.48)
+		)
+		(stroke
+			(width 0)
+			(type default)
+		)
+	)
+	(wire
+		(pts
 			(xy 31.75 39.37) (xy 34.29 39.37)
 		)
@@
 	(wire
 		(pts
+			(xy 43.18 17.78) (xy 43.18 19.05)
+		)
+		(stroke
+			(width 0)
+			(type default)
+		)
+	)
+	(wire
+		(pts
 			(xy 115.57 34.29) (xy 127 34.29)
 		)
@@
 	(wire
 		(pts
+			(xy 43.18 30.48) (xy 54.61 30.48)
+		)
+		(stroke
+			(width 0)
+			(type default)
+		)
+	)
+	(wire
+		(pts
 			(xy 149.86 29.21) (xy 152.4 29.21)
 		)
@@
 	(wire
 		(pts
-			(xy 48.26 30.48) (xy 54.61 30.48)
-		)
-		(stroke
-			(width 0)
-			(type default)
-		)
-	)
-	(wire
-		(pts
 			(xy 48.26 33.02) (xy 54.61 33.02)
 		)
@@
 		)
 	)
-	(global_label "SPI_M0SI"
+	(global_label "SPI_MOSI"
 		(shape input)
 		(at 48.26 29.21 180)
@@
 		)
 		(property "Intersheetrefs" "${INTERSHEET_REFS}"
-			(at 43.6551 29.21 0)
+			(at 43.6067 29.21 0)
 			(effects
 				(font
@@
 	(global_label "SPI_CLK"
 		(shape input)
-		(at 48.26 30.48 180)
+		(at 43.18 17.78 90)
 		(fields_autoplaced yes)
 		(effects
@@
 				(size 0.508 0.508)
 			)
-			(justify right)
+			(justify left)
 		)
 		(property "Intersheetrefs" "${INTERSHEET_REFS}"
-			(at 44.018 30.48 0)
+			(at 43.18 13.538 90)
 			(effects
 				(font
 					(size 1.27 1.27)
 				)
-				(justify right)
+				(justify left)
 				(hide yes)
 			)
@@
 			)
 		)
-		(property "Footprint" "MT7628:MT7628_footprint"
+		(property "Footprint" "Library:MT7628_footprint"
 			(at 62.23 27.94 0)
 			(effects
@@
 			)
 		)
-		(property "Footprint" "MT7628:MT7628_footprint"
+		(property "Footprint" "Library:MT7628_footprint"
 			(at 163.83 43.18 0)
 			(effects
@@
 	)
 	(symbol
+		(lib_id "MT7688AN_Reset-altium-import:root_2_Res1_Miscellaneous Devices.SchLib")
+		(at 45.72 21.59 90)
+		(unit 1)
+		(exclude_from_sim no)
+		(in_bom yes)
+		(on_board yes)
+		(dnp no)
+		(property "Reference" "R11"
+			(at 42.418 26.924 0)
+			(effects
+				(font
+					(size 1.27 1.27)
+				)
+				(justify left bottom)
+			)
+		)
+		(property "Value" "22"
+			(at 42.418 29.718 0)
+			(effects
+				(font
+					(size 1.27 1.27)
+				)
+				(justify left bottom)
+				(hide yes)
+			)
+		)
+		(property "Footprint" "Resistor_SMD:R_0402_1005Metric"
+			(at 45.72 21.59 0)
+			(effects
+				(font
+					(size 1.27 1.27)
+				)
+				(hide yes)
+			)
+		)
+		(property "Datasheet" ""
+			(at 45.72 21.59 0)
+			(effects
+				(font
+					(size 1.27 1.27)
+				)
+				(hide yes)
+			)
+		)
+		(property "Description" "Resistor"
+			(at 45.72 21.59 0)
+			(effects
+				(font
+					(size 1.27 1.27)
+				)
+				(hide yes)
+			)
+		)
+		(property "PUBLISHED" "8-Jun-2000"
+			(at 42.418 29.718 0)
+			(effects
+				(font
+					(size 1.27 1.27)
+				)
+				(justify left bottom)
+				(hide yes)
+			)
+		)
+		(property "LATESTREVISIONDATE" "17-Jul-2002"
+			(at 42.418 29.718 0)
+			(effects
+				(font
+					(size 1.27 1.27)
+				)
+				(justify left bottom)
+				(hide yes)
+			)
+		)
+		(property "LATESTREVISIONNOTE" "Re-released for DXP Platform."
+			(at 42.418 29.718 0)
+			(effects
+				(font
+					(size 1.27 1.27)
+				)
+				(justify left bottom)
+				(hide yes)
+			)
+		)
+		(property "PACKAGEREFERENCE" "AXIAL-0.3"
+			(at 42.418 29.718 0)
+			(effects
+				(font
+					(size 1.27 1.27)
+				)
+				(justify left bottom)
+				(hide yes)
+			)
+		)
+		(property "PUBLISHER" "Altium Limited"
+			(at 42.418 29.718 0)
+			(effects
+				(font
+					(size 1.27 1.27)
+				)
+				(justify left bottom)
+				(hide yes)
+			)
+		)
+		(property "PACKAGEDESCRIPTION" "Axial Device, Thru-Hole; 2 Leads; 0.3 in Pin Spacing"
+			(at 42.418 29.718 0)
+			(effects
+				(font
+					(size 1.27 1.27)
+				)
+				(justify left bottom)
+				(hide yes)
+			)
+		)
+		(property "ALTIUM_VALUE" "22¦¸"
+			(at 46.482 26.924 0)
+			(effects
+				(font
+					(size 1.27 1.27)
+				)
+				(justify left bottom)
+				(hide yes)
+			)
+		)
+		(property "LCSC" "C25092"
+			(at 45.72 21.59 0)
+			(effects
+				(font
+					(size 1.27 1.27)
+				)
+				(hide yes)
+			)
+		)
+		(pin "2"
+		)
+		(pin "1"
+		)
+		(instances
+			(project "mt7628v1"
+				(path "/144686d4-2b77-460c-9924-cc86faff7e9d/218ba002-e319-46e9-a80e-651bdbb44c2c"
+					(reference "R11")
+					(unit 1)
+				)
+			)
+		)
+	)
+	(symbol
 		(lib_id "Device:C")
 		(at 88.9 93.98 0)
@@
 			)
 		)
-		(property "Footprint" "MT7628:MT7628_footprint"
+		(property "Footprint" "Library:MT7628_footprint"
 			(at 124.46 99.06 0)
 			(effects

Commit message: final_all_router by asif
Parts:
- removed R15, R16: 10K/1% NC, Resistor_SMD:R_0402_1005Metric, symbol Device:R
- U2: value ~ -> MT7628NN; LCSC (none) -> C2762437
Connections:
- net WDT_RST: now reaches R38.2, U2.137 (WDT_RST_N)
- net USB_DP+: now reaches R18.2, U2.61 (USB_DP)
- net LINK3: now reaches U2.140 (AVDD33_TX_P1234_2)
- net LINK2: now reaches U2.141 (EPHY_LED2_N_JTMS)
- net USB_DP-: now reaches R19.2, U2.62 (USB_DM)
- net EPH_LED0_N renamed LINK0
- net EPH_LED1_N renamed LINK1
- net I2S_D0 renamed I2S_SDO
- net I2S_DI renamed I2S_SDI
- net PORST_N renamed CPURST_N
- net PWM_CH0 renamed RXN2
- net PWM_CH1 renamed RXP2
- net RXIN1 renamed TXP1
- net RXIP1 renamed TXN1
- net SD_CD renamed RXP3
- net SD_CLK renamed RXN4
- net SD_CMD renamed RXP4
- net SD_D0 renamed TXP3
- net SD_D1 renamed TXN3
- net SD_D2 renamed TXP4
- net SD_D3 renamed TXN4
- net SD_WP renamed RXN3
- net TXON1 renamed RXP1
- net TXOP1 renamed RXN1
- net UART_RXD2 renamed TXN2
- net UART_TXD2 renamed TXP2
- net WIFI_RESET renamed LINK4
- no-connect marks 9 -> 7
Other:
- moved on the sheet: R18, R19, R38
