File: RF_Front_End.kicad_sch (KiCad schematic)
At the start: 1 part

Commit message: updated aux
Parts:
- U2: footprint (none) -> MT7628:MT7628_footprint
Other:
- moved on the sheet: U2A
Changed lines of the file:
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@@
 	(symbol
 		(lib_id "mt7628_222:MT7628_*")
-		(at 48.26 45.72 0)
+		(at 96.52 48.26 0)
 		(unit 1)
 		(exclude_from_sim no)
@@
 		(dnp no)
 		(property "Reference" "U2"
-			(at 48.006 37.846 0)
+			(at 96.266 40.386 0)
 			(effects
 				(font
@@
 		)
 		(property "Value" "~"
-			(at 48.895 38.1 0)
+			(at 97.155 40.64 0)
 			(effects
 				(font
@@
 			)
 		)
-		(property "Footprint" ""
-			(at 48.26 45.72 0)
+		(property "Footprint" "MT7628:MT7628_footprint"
+			(at 96.52 48.26 0)
 			(effects
 				(font
@@
 		)
 		(property "Datasheet" ""
-			(at 48.26 45.72 0)
+			(at 96.52 48.26 0)
 			(effects
 				(font
@@
 		)
 		(property "Description" ""
-			(at 48.26 45.72 0)
+			(at 96.52 48.26 0)
 			(effects
 				(font

Commit message: init_sch
Parts:
- added C41: 10uf/6.3v, symbol Device:C
- added C42, C52, C59, C62: 10pf/50v, symbol Device:C
- added C43, C45, C47, C48, C51, C61, C66, C68: 1uf/6.3v, symbol Device:C
- added C44, C46, C50, C60, C64, C65, C67, C69: 100pf/50v, symbol Device:C
- added C49: 10uf/6.3v NC, symbol Device:C
- added C53, C62: 1.2pf/50v, symbol Device:C
- added C54, C56: 2pf/50v, symbol Device:C
- added C55: 9pf/50v, symbol Device:C
- added C57, C58: 1.8Pf/50v, symbol Device:C
- added C63: 1.3pf/50v, symbol Device:C
- added L2, L3: 10nh, symbol Device:L
- added L4, L9: 2.7nh, symbol Device:L
- added L5, L7, L8: 2nh, symbol Device:L
- added L6: 1.2nh, symbol Device:L
- added R20, R21: 0, symbol Device:R
- added RF1: ANT_SHAFT_SEAT, easyeda2kicad:IPEX-SMD_4P-L2.6-W2.6_C9900016457, symbol testeda:ANT_SHAFT_SEAT
- added Y1: Crystal_40Mhz, easyeda2kicad:CRYSTAL-SMD_4P-L3.2-W2.5-BL, symbol Device:Crystal_GND23
Connections:
- net GND: now reaches U2.1 (AVSS33_RF_1)
- net GND: now also U2.10 (AVSS33_RF_4), U2.13 (AVSS33_RF_5), U2.152 (AVSS33_XTAL), U2.156 (WF0_LNA_EXT), U2.2 (AVSS33_RF_2), C41.2, C42.2, C43.2, C44.2, C45.2, C46.2, C47.2, C48.2, C49.2, C50.2, C51.2, C54.2, C56.2, C57.2, C58.2, C60.2, C61.2, C62.1, C62.2, C63.2, C64.2, C65.2, C66.2, C67.2, C68.2, C69.2, L4.1, RF1.1, RF1.2, Y1.2, Y1.3, Y1.4
- net 3.3V_RF: now reaches U2.14 (AVDD33_WF1_TX)
- net 3.3V_RF: now also U2.149 (AVDD33_WF_RFDIG), U2.15 (AVDD33_WF1_TRX), U2.150 (AVDD33_XTAL), U2.155 (AVDD33_WF0_TRX), U2.8 (AVDD33_WF0_TX), C44.1, C45.1, C48.1, C49.1, C50.1, C51.1, C60.1, C61.1, C64.1, C65.1, C66.1, C67.1, C68.1, C69.1, L2.1, L3.1, R20.2, R21.1
- net at U2.151 (XTALIN): now also C62.1, C63.1, Y1.1
- net WF_SX_3V3_IN: now reaches U2.154 (AVDD33_WF_SX)
- net WF_SX_3V3_IN: now also C46.1, C47.1, R21.2
- net at U2.3 (WF0_RFION_1): now also U2.4 (WF0_RFION_2), C56.1, L3.2, L8.1
- net at U2.5 (WF0_RFIOP_1): now also U2.6 (WF0_RFIOP_2), C54.1, L2.2, L5.1
- new net: C59.1, L8.2
- new net: C52.1, L5.2
- new net: C52.2, C53.1, L4.2
- new net: C59.2, C62.2, L9.1
- new net 3.3VD: C41.1, C42.1, C43.1, R20.1
- new net RFOUT_G0: C55.2, C57.1, L6.2, L7.1
- new net RFOUT_G0_L: C53.2, C55.1, L6.1, L9.2
- new net WF0_iPA: C58.1, L7.2, RF1.3
- no-connect marks 0 -> 5

Commit message: updated
Parts:
- removed C62: 10pf/50v, symbol Device:C
- C41, C49: footprint (none) -> Capacitor_SMD:C_0603_1608Metric; LCSC (none) -> C1691
- C42, C52, C59: footprint (none) -> Capacitor_SMD:C_0402_1005Metric; LCSC (none) -> C32949
- C43, C45, C47, C48, C51, C61, C66, C68: footprint (none) -> Capacitor_SMD:C_0402_1005Metric; LCSC (none) -> C15684
- C44, C46, C50, C60, C64, C65, C67, C69: footprint (none) -> Capacitor_SMD:C_0402_1005Metric; LCSC (none) -> C1546
- C53, C62: footprint (none) -> Capacitor_SMD:C_0402_1005Metric; LOSC (none) -> C1551
- C54, C56: footprint (none) -> Capacitor_SMD:C_0402_1005Metric; LOSC (none) -> C1523
- C55: footprint (none) -> Capacitor_SMD:C_0402_1005Metric; LOSC (none) -> C1580
- C57, C58: footprint (none) -> Capacitor_SMD:C_0402_1005Metric; LOSC (none) -> C1553
- C63: footprint (none) -> Capacitor_SMD:C_0402_1005Metric; LCSC (none) -> C88880
- L2, L3: footprint (none) -> Inductor_SMD:L_0402_1005Metric; LCSC (none) -> C21585
- L4, L9: footprint (none) -> Inductor_SMD:L_0402_1005Metric; LCSC (none) -> C76770
- L5, L7, L8: footprint (none) -> Inductor_SMD:L_0402_1005Metric; LCSC (none) -> C18216
- L6: footprint (none) -> Inductor_SMD:L_0402_1005Metric; LCSC (none) -> C77105
- R20, R21: footprint (none) -> Resistor_SMD:R_0402_1005Metric; LCSC (none) -> C17168
- RF1: LCSC (none) -> C9900016457; LCSC Part C9900016457 -> (none)

Commit message: f_ver
Parts:
- C49: now not fitted; now left out of the parts list
- U2: footprint MT7628:MT7628_footprint -> Library:MT7628_footprint
Changed lines of the file:
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@@
 			)
 		)
-		(property "Footprint" "MT7628:MT7628_footprint"
+		(property "Footprint" "Library:MT7628_footprint"
 			(at 96.52 48.26 0)
 			(effects
@@
 		(at 176.53 41.91 0)
 		(unit 1)
-		(exclude_from_sim no)
-		(in_bom yes)
-		(on_board yes)
-		(dnp no)
+		(exclude_from_sim yes)
+		(in_bom no)
+		(on_board no)
+		(dnp yes)
 		(property "Reference" "C49"
 			(at 176.784 39.878 0)

Commit message: final_all_router by asif
Parts:
- removed C68: 1uf/6.3v, Capacitor_SMD:C_0402_1005Metric, symbol Device:C
- added C100, C101: 10pf/50v, Capacitor_SMD:C_0402_1005Metric, symbol Device:C
- added C102, C103: 1.2pf/50v, Capacitor_SMD:C_0402_1005Metric, symbol Device:C
- added C104: 9pf/50v, Capacitor_SMD:C_0402_1005Metric, symbol Device:C
- added C105, C106: 1.8Pf/50v, Capacitor_SMD:C_0402_1005Metric, symbol Device:C
- added C79, C80: 2pf/50v, Capacitor_SMD:C_0402_1005Metric, symbol Device:C
- added C81, C82: 1uf/6.3v, Capacitor_SMD:C_0402_1005Metric, symbol Device:C
- added C83: 100pf/50v, Capacitor_SMD:C_0402_1005Metric, symbol Device:C
- added L10, L12: 10nh, Inductor_SMD:L_0402_1005Metric, symbol Device:L
- added L13, L14, L18: 2nh, Inductor_SMD:L_0402_1005Metric, symbol Device:L
- added L15, L16: 2.7nh, Inductor_SMD:L_0402_1005Metric, symbol Device:L
- added L17: 1.2nh, Inductor_SMD:L_0402_1005Metric, symbol Device:L
- added RF2: ANT_SHAFT_SEAT, easyeda2kicad:IPEX-SMD_4P-L2.6-W2.6_C9900016457, symbol testeda:ANT_SHAFT_SEAT
- C53, C62: LCSC (none) -> C1551; LOSC C1551 -> (none)
- C54, C56: LCSC (none) -> C1523; LOSC C1523 -> (none)
- C55: LCSC (none) -> C1580; LOSC C1580 -> (none)
- C57, C58: LCSC (none) -> C1553; LOSC C1553 -> (none)
- U2: value ~ -> MT7628NN; LCSC (none) -> C2762437
Connections:
- net 3.3V_RF: now also C81.1, C82.1, C83.1, L10.1, L12.1
- net GND: now also U2.7 (AVSS33_RF_3), C102.1, C105.2, C106.2, C79.2, C80.1, C81.2, C82.2, C83.2, L15.1, RF2.1, RF2.2
- net WF1_RF1ON: now reaches U2.11 (WF1_RFION)
- net WF1_RF1ON: now also C80.2, L12.2, L14.1
- net WF1_RF1OP: now reaches U2.12 (WF1_RFIOP)
- net WF1_RF1OP: now also C79.1, L10.2, L13.1
- new net: C101.2, C102.2, L16.1
- new net: C103.2, C104.1, L16.2, L17.1
- new net: C104.2, C105.1, L17.2, L18.1
- new net: C106.1, L18.2, RF2.3
- new net: C100.2, C103.1, L15.2
- new net: C100.1, L13.2
- new net: C101.1, L14.2
- no-connect marks 5 -> 2
