File: config.kicad_sch (KiCad schematic)
At the start: 0 parts

Commit message: init_sch
Parts:
- added R1, R2, R25, R26, R27, R28, R29, R3, R30, R31, R4, R5, R6, R7: 4.7k, Resistor_SMD:R_0402_1005Metric, symbol Config-altium-import:root_0_Res1_Miscellaneous Devices.SchLib
Connections:
- new net 3.3VD: R2.1, R25.1, R26.1, R28.1, R3.1, R31.1, R5.1
- new net GND: R1.1, R27.1, R29.1, R30.1, R4.1, R6.1, R7.1
- new net I2S_DO: R31.2, R7.2
- new net PERST_N: R3.2, R30.2
- new net SPI_CLK: R2.2, R4.2
- new net SPI_CS1: R5.2, R6.2
- new net SPI_MOSI: R1.2, R25.2
- new net UART_TXD0: R28.2, R29.2
- new net UART_TXD1: R26.2, R27.2
Other:
- note added: "010: Boot from XTAL (Boot from SPI 3-Byte Addr ) ×î´óÖ§³Ö128Mbit"
- note added: "011: Boot from XTAL (Boot from SPI 4-Byte Addr) ×î´óÖ§³Ö512Mbit"
- note added: "0: 25MHz DIP"
- note added: "0: DDR2"
- note added: "0: JTAG_MODE"
- note added: "0: Normal"
- note added: "1: 40MHz SMD"
- note added: "1: DDR1"
- note added: "1: EPHY_LED"
- note added: "1: Test mode"

Commit message: updated
Changed lines of the file:
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@@
-	(wire
-		(pts
-			(xy 236.22 132.08) (xy 167.64 132.08)
-		)
-		(stroke
-			(width 0)
-			(type default)
-		)
-	)
 	(wire
 		(pts
@@
 	(wire
 		(pts
-			(xy 236.22 66.04) (xy 236.22 132.08)
-		)
-		(stroke
-			(width 0)
-			(type default)
-		)
-	)
-	(wire
-		(pts
 			(xy 81.28 78.74) (xy 91.44 78.74)
 		)
@@
 	(wire
 		(pts
-			(xy 167.64 132.08) (xy 167.64 66.04)
-		)
-		(stroke
-			(width 0)
-			(type default)
-		)
-	)
-	(wire
-		(pts
 			(xy 81.28 86.36) (xy 91.44 86.36)
 		)
@@
 		(pts
 			(xy 63.5 121.92) (xy 71.12 121.92)
-		)
-		(stroke
-			(width 0)
-			(type default)
-		)
-	)
-	(wire
-		(pts
-			(xy 167.64 66.04) (xy 236.22 66.04)
 		)
 		(stroke
@@
 		)
 	)
-	(hierarchical_label "SPI_CS1"
-		(shape bidirectional)
+	(global_label "PERST_N"
+		(shape input)
+		(at 83.82 58.42 180)
+		(fields_autoplaced yes)
+		(effects
+			(font
+				(size 1.27 1.27)
+			)
+			(justify right)
+		)
+		(property "Intersheetrefs" "${INTERSHEET_REFS}"
+			(at 72.6706 58.42 0)
+			(effects
+				(font
+					(size 1.27 1.27)
+				)
+				(justify right)
+				(hide yes)
+			)
+		)
+	)
+	(global_label "SPI_MOSI"
+		(shape input)
+		(at 83.82 38.1 180)
+		(fields_autoplaced yes)
+		(effects
+			(font
+				(size 1.27 1.27)
+			)
+			(justify right)
+		)
+		(property "Intersheetrefs" "${INTERSHEET_REFS}"
+			(at 72.1867 38.1 0)
+			(effects
+				(font
+					(size 1.27 1.27)
+				)
+				(justify right)
+				(hide yes)
+			)
+		)
+	)
+	(global_label "UART_TXD0"
+		(shape input)
+		(at 83.82 53.34 180)
+		(fields_autoplaced yes)
+		(effects
+			(font
+				(size 1.27 1.27)
+			)
+			(justify right)
+		)
+		(property "Intersheetrefs" "${INTERSHEET_REFS}"
+			(at 70.5539 53.34 0)
+			(effects
+				(font
+					(size 1.27 1.27)
+				)
+				(justify right)
+				(hide yes)
+			)
+		)
+	)
+	(global_label "I2S_DO"
+		(shape input)
+		(at 83.82 33.02 180)
+		(fields_autoplaced yes)
+		(effects
+			(font
+				(size 1.27 1.27)
+			)
+			(justify right)
+		)
+		(property "Intersheetrefs" "${INTERSHEET_REFS}"
+			(at 74.2429 33.02 0)
+			(effects
+				(font
+					(size 1.27 1.27)
+				)
+				(justify right)
+				(hide yes)
+			)
+		)
+	)
+	(global_label "UART_TXD1"
+		(shape input)
+		(at 83.82 63.5 180)
+		(fields_autoplaced yes)
+		(effects
+			(font
+				(size 1.27 1.27)
+			)
+			(justify right)
+		)
+		(property "Intersheetrefs" "${INTERSHEET_REFS}"
+			(at 70.5539 63.5 0)
+			(effects
+				(font
+					(size 1.27 1.27)
+				)
+				(justify right)
+				(hide yes)
+			)
+		)
+	)
+	(global_label "SPI_CLK"
+		(shape input)
+		(at 83.82 43.18 180)
+		(fields_autoplaced yes)
+		(effects
+			(font
+				(size 1.27 1.27)
+			)
+			(justify right)
+		)
+		(property "Intersheetrefs" "${INTERSHEET_REFS}"
+			(at 73.2148 43.18 0)
+			(effects
+				(font
+					(size 1.27 1.27)
+				)
+				(justify right)
+				(hide yes)
+			)
+		)
+	)
+	(global_label "SPI_CS1"
+		(shape input)
 		(at 83.82 48.26 180)
+		(fields_autoplaced yes)
 		(effects
 			(font
@@
 			(justify right)
 		)
-	)
-	(hierarchical_label "UART_TXD1"
-		(shape bidirectional)
-		(at 83.82 63.5 180)
-		(effects
-			(font
-				(size 1.27 1.27)
-			)
-			(justify right)
-		)
-	)
-	(hierarchical_label "SPI_MOSI"
-		(shape bidirectional)
-		(at 83.82 38.1 180)
-		(effects
-			(font
-				(size 1.27 1.27)
-			)
-			(justify right)
-		)
-	)
-	(hierarchical_label "I2S_DO"
-		(shape bidirectional)
-		(at 83.82 33.02 180)
-		(effects
-			(font
-				(size 1.27 1.27)
-			)
-			(justify right)
-		)
-	)
-	(hierarchical_label "UART_TXD0"
-		(shape bidirectional)
-		(at 83.82 53.34 180)
-		(effects
-			(font
-				(size 1.27 1.27)
-			)
-			(justify right)
-		)
-	)
-	(hierarchical_label "PERST_N"
-		(shape bidirectional)
-		(at 83.82 58.42 180)
-		(effects
-			(font
-				(size 1.27 1.27)
-			)
-			(justify right)
-		)
-	)
-	(hierarchical_label "SPI_CLK"
-		(shape bidirectional)
-		(at 83.82 43.18 180)
-		(effects
-			(font
-				(size 1.27 1.27)
-			)
-			(justify right)
-		)
-	)
+		(property "Intersheetrefs" "${INTERSHEET_REFS}"
+			(at 73.0939 48.26 0)
+			(effects
+				(font
+					(size 1.27 1.27)
+				)
+				(justify right)
+				(hide yes)
+			)
+		)
+	)

Commit message: f_ver
Parts:
- R31: LCSC (none) -> NC
- R7: LCSC (none) -> C25900
Changed lines of the file:
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@@
+			)
+		)
+		(property "LCSC" "C25900"
+			(at 73.66 147.32 0)
+			(effects
+				(font
+					(size 1.27 1.27)
+				)
+				(hide yes)
 			)
 		)
@@
 			)
 		)
+		(property "LCSC" "NC"
+			(at 73.66 139.7 0)
+			(effects
+				(font
+					(size 1.27 1.27)
+				)
+				(hide yes)
+			)
+		)

Commit message: final_all_router by asif
Parts:
- R27: LCSC C25900 -> NC
- R28: LCSC (none) -> NC
Changed lines of the file:
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@@
 			)
 		)
-		(property "LCSC" "C25900"
+		(property "LCSC" "NC"
 			(at 73.66 83.82 0)
 			(effects
@@
 			)
 		)
-		(property "LCSC" ""
+		(property "LCSC" "NC"
 			(at 73.66 99.06 0)
 			(effects
