File: ddr_cfg.kicad_sch (KiCad schematic)
At the start: 0 parts

Commit message: init_sch
Parts:
- added C1, C15, C16, C19, C2, C4: 100nf/16v, 0402_C, symbol DDR2_CFG-altium-import:root_1_Cap_Miscellaneous Devices.SchLib
- added C3: 4.7uf/6.3v, 0603_C, symbol DDR2_CFG-altium-import:root_3_Cap2_Miscellaneous Devices.SchLib
- added R10: 100/1%, 0402_R, symbol DDR2_CFG-altium-import:root_1_Res1_Miscellaneous Devices.SchLib
- added R32: 10k/1%, 0402_R, symbol DDR2_CFG-altium-import:root_2_Res1_Miscellaneous Devices.SchLib
- added R33: 1k/1%, 0402_R, symbol DDR2_CFG-altium-import:root_1_Res1_Miscellaneous Devices.SchLib
- added R8: 1K/1%, 0402_R, symbol DDR2_CFG-altium-import:root_1_Res1_Miscellaneous Devices.SchLib
- added R9: 100nf/1%, 0402_R, symbol DDR2_CFG-altium-import:root_1_Res1_Miscellaneous Devices.SchLib
- added U1: W9751G6KB, wbga-84, symbol DDR2_CFG-altium-import:root_0_W9751G6KB_MT7688_PCBProject.SCHLIB
Connections:
- new net CLK_N: R10.1, U1.K8 (CK_N)
- new net CLK_P: R10.2, U1.J8 (CK_P)
- new net DDR_BA0: U1.L2 (BA0)
- new net DDR_BA1: U1.L3 (BA1)
- new net DDR_BA2: U1.L1 (BA2)
- new net DDR_CASN: U1.L7 (~{CAS})
- new net DDR_CSN: U1.L8 (~{CS})
- new net DDR_IO_1V8_MT7688: C1.2, C15.2, C16.2, C19.2, C3.1, C4.2, R32.1, R8.2, U1.A1 (VDD), U1.A9 (VDDQ), U1.C1 (VDDQ), U1.C3 (VDDQ), U1.C7 (VDDQ), U1.C9 (VDDQ), U1.E1 (VDD), U1.E9 (VDDQ), U1.G1 (VDDQ), U1.G3 (VDDQ), U1.G7 (VDDQ), U1.G9 (VDDQ), U1.J1 (VDDL), U1.J9 (VDD), U1.M9 (VDD), U1.R1 (VDD)
- new net DDR_MCKE: U1.K2 (CKE)
- new net DDR_MDQM0: U1.F3 (LDM)
- new net DDR_MDQM1: U1.B3 (UDM)
- new net DDR_MDQS0: U1.F7 (LDQS_P)
- new net DDR_MDQS1: U1.B7 (UDQS_P)
- new net DDR_MODT: R32.2, R33.2, U1.K9 (ODT)
- new net DDR_RASN: U1.K7 (~{RAS})
- new net DDR_VREF: C1.1, C2.2, R8.1, R9.2, U1.J2 (VREF)
- new net DDR_WEN: U1.K3 (~{WE})
- new net GND: C15.1, C16.1, C19.1, C2.1, C3.2, C4.1, R33.1, R9.1, U1.A3 (VSS), U1.A7 (VSSQ), U1.B2 (VSSQ), U1.B8 (VSSQ), U1.D2 (VSSQ), U1.D8 (VSSQ), U1.E3 (VSS), U1.E7 (VSSQ), U1.F2 (VSSQ), U1.F8 (VSSQ), U1.H2 (VSSQ), U1.H8 (VSSQ), U1.J3 (VSS), U1.J7 (VSSDL), U1.N1 (VSS), U1.P9 (VSS)
- new net MADDR0: U1.M8 (A0)
- new net MADDR1: U1.M3 (A1)
- new net MADDR10: U1.M2 (A10)
- new net MADDR11: U1.P7 (A11)
- new net MADDR12: U1.R2 (A12)
- new net MADDR13: U1.R8 (A13(2GB))
- new net MADDR2: U1.M7 (A2)
- new net MADDR3: U1.N2 (A3)
- new net MADDR4: U1.N8 (A4)
- new net MADDR5: U1.N3 (A5)
- new net MADDR6: U1.N7 (A6)
- new net MADDR7: U1.P2 (A7)
- new net MADDR8: U1.P8 (A8)
- new net MADDR9: U1.P3 (A9)
- new net MDATA0: U1.G8 (DQ0)
- new net MDATA1: U1.G2 (DQ1)
- new net MDATA10: U1.D7 (DQ10)
- new net MDATA11: U1.D3 (DQ11)
- new net MDATA12: U1.D1 (DQ12)
- new net MDATA13: U1.D9 (DQ13)
- new net MDATA14: U1.B1 (DQ14)
- new net MDATA15: U1.B9 (DQ15)
- new net MDATA2: U1.H7 (DQ2)
- new net MDATA3: U1.H3 (DQ3)
- new net MDATA4: U1.H1 (DQ4)
- new net MDATA5: U1.H9 (DQ5)
- new net MDATA6: U1.F1 (DQ6)
- new net MDATA7: U1.F9 (DQ7)
- new net MDATA8: U1.C8 (DQ8)
- new net MDATA9: U1.C2 (DQ9)
- no-connect marks 0 -> 6
Other:
- note added: "Place close to the DDR2"

Commit message: updated
Parts:
- C1, C2, C4: footprint 0402_C -> Capacitor_SMD:C_0402_1005Metric; LCSC (none) -> C1525
- C3: footprint 0603_C -> Capacitor_SMD:C_0603_1608Metric; LCSC (none) -> C8032
- C5: renamed from C15; footprint 0402_C -> Capacitor_SMD:C_0402_1005Metric; LCSC (none) -> C1525
- C6: renamed from C16; footprint 0402_C -> Capacitor_SMD:C_0402_1005Metric; LCSC (none) -> C1525
- C7: renamed from C19; footprint 0402_C -> Capacitor_SMD:C_0402_1005Metric; LCSC (none) -> C1525
- R10: footprint 0402_R -> Resistor_SMD:R_0402_1005Metric; LCSC (none) -> C25076
- R32: footprint 0402_R -> Resistor_SMD:R_0402_1005Metric; LCSC (none) -> C25744
- R33, R8, R9: footprint 0402_R -> Resistor_SMD:R_0402_1005Metric; LCSC (none) -> C11702
- U1: value W9751G6KB -> W9725G6KB-25; footprint wbga-84 -> easyeda2kicad:WBGA-84_L12.5-W8.0-P0.80-TL_WINBOND_W9725G6KB; LCSC (none) -> C571266
Connections:
- net DDR_IO_1V8_MT7688 renamed DDR_IO_1V8_MT7628

Commit message: f_ver
Changed lines of the file:
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@@
-	(wire
-		(pts
-			(xy 196.85 26.67) (xy 196.85 88.9)
-		)
-		(stroke
-			(width 0)
-			(type default)
-		)
-	)
 	(wire
 		(pts
@@
 	(wire
 		(pts
-			(xy 196.85 88.9) (xy 266.7 88.9)
-		)
-		(stroke
-			(width 0)
-			(type default)
-		)
-	)
-	(wire
-		(pts
-			(xy 266.7 26.67) (xy 196.85 26.67)
-		)
-		(stroke
-			(width 0)
-			(type default)
-		)
-	)
-	(wire
-		(pts
 			(xy 127 41.91) (xy 129.54 41.91)
 		)
@@
 		)
 		(stroke
-			(width 0)
-			(type default)
-		)
-	)
-	(wire
-		(pts
-			(xy 266.7 88.9) (xy 266.7 26.67)
-		)
-		(stroke

Commit message: final_all_router by asif
Parts:
- U1: value W9725G6KB-25 -> W971GG6SB25I; footprint easyeda2kicad:WBGA-84_L12.5-W8.0-P0.80-TL_WINBOND_W9725G6KB -> easyeda2kicad:WBGA-84_L12.5-W8.0-P0.80-TL_W9751G6KB; LCSC C571266 -> C191947
Connections:
- net MADDR13: no longer names the net of U1.R8 (A13(2GB))
- no-connect marks 6 -> 7
Changed lines of the file:
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@@
 	)
 	(no_connect
+		(at 78.74 97.79)
+	)
+	(no_connect
 		(at 157.48 137.16)
 	)
@@
 	)
 	(bus_entry
-		(at 58.42 95.25)
-		(size 2.54 2.54)
-		(stroke
-			(width 0)
-			(type default)
-		)
-	)
-	(bus_entry
 		(at 58.42 69.85)
 		(size 2.54 2.54)
@@
 		)
 	)
-	(wire
-		(pts
-			(xy 60.96 97.79) (xy 78.74 97.79)
-		)
-		(stroke
-			(width 0)
-			(type default)
-		)
-	)
 	(bus
 		(pts
@@
 		)
 	)
-	(label "MADDR13"
-		(at 63.5 97.79 0)
-		(effects
-			(font
-				(size 1.27 1.27)
-			)
-			(justify left bottom)
-		)
-	)
 	(label "DDR_CASN"
 		(at 55.88 135.89 0)
@@
 		)
 	)
-	(label "MADDR[0..13]"
+	(label "MADDR[0..12]"
 		(at 40.64 54.61 0)
 		(effects
@@
 			)
 		)
-		(property "Value" "W9725G6KB-25"
+		(property "Value" "W971GG6SB25I"
 			(at 157.988 58.42 0)
 			(effects
@@
 			)
 		)
-		(property "Footprint" "easyeda2kicad:WBGA-84_L12.5-W8.0-P0.80-TL_WINBOND_W9725G6KB"
+		(property "Footprint" "easyeda2kicad:WBGA-84_L12.5-W8.0-P0.80-TL_W9751G6KB"
 			(at 86.36 151.13 0)
 			(effects
@@
 			)
 		)
-		(property "LCSC" "C571266"
+		(property "LCSC" "C191947"
 			(at 86.36 151.13 0)
 			(effects
