File: ddr_if.kicad_sch (KiCad schematic)
At the start: 1 part

Commit message: updated aux
Parts:
- added C8: 1uf/6.3v, symbol Device:C
- U2: footprint (none) -> MT7628:MT7628_footprint
Connections:
- net DDR_BA0: now reaches U2.100 (MBA0)
- net DDR_BA2: now reaches U2.101 (MBA2)
- net DDR_WEN: now reaches U2.102 (MW_E)
- net DDR_MCKE: now reaches U2.103 (MCKE)
- net DDR_VREF: now reaches U2.104 (DDR_IO_VREF_2)
- net DDR_VREF: now also U2.90 (DDR_IO_VREF_1), C8.1
- net MDATA3: now reaches U2.105 (MD3)
- net MDATA4: now reaches U2.106 (MD4)
- net MDATA1: now reaches U2.107 (MD1)
- net DDR_MDQM0: now reaches U2.108 (MDQM0)
- net MDATA6: now reaches U2.109 (MD6)
- net MDATA11: now reaches U2.110 (MD11)
- net MDATA12: now reaches U2.111 (MD12)
- net MDATA9: now reaches U2.112 (MD9)
- net DDR_MDQS0: now reaches U2.113 (MDQS0)
- net MDATA14: now reaches U2.114 (MD14)
- net GND: now reaches U2.115 (DDR_IO_VSS_2)
- net GND: now also U2.63 (DDR_IO_VSS_1), C8.2
- net DDR_IO_1V8_MT7688: now reaches U2.116 (DDR_IO_1V8D_3)
- net DDR_IO_1V8_MT7688: now also U2.79 (DDR_IO_1V8D_1), U2.98 (DDR_IO_1V8D_2)
- net DDR_MDQM1: now reaches U2.64 (MDQM1)
- net MDATA15: now reaches U2.65 (MD15)
- net MDATA8: now reaches U2.66 (MD8)
- net MDATA13: now reaches U2.67 (MD13)
- net MDATA10: now reaches U2.68 (MD10)
- net MDATA2: now reaches U2.69 (MD2)
- net MDATA7: now reaches U2.70 (MD7)
- net MDATA0: now reaches U2.71 (MD0)
- net DDR_MDQS1: now reaches U2.72 (MDQS1)
- net MDATA5: now reaches U2.73 (MD5)
- net DDR_MODT: now reaches U2.74 (MODT)
- net DDR_CASN: now reaches U2.75 (MCAS)
- net CLK_N: now reaches U2.76 (MCK_N)
- net CLK_P: now reaches U2.77 (MCK_P)
- net DDR_CSN: now reaches U2.78 (MCS)
- net MADDR0: now reaches U2.80 (MA0)
- net DDR_RASN: now reaches U2.81 (MRAS)
- net MADDR4: now reaches U2.82 (MA4)
- net MADDR13: now reaches U2.83 (MA13)
- net MADDR8: now reaches U2.84 (MA8)
- net MADDR11: now reaches U2.85 (MA11)
- net MADDR6: now reaches U2.86 (MA6)
- net MADDR2: now reaches U2.87 (MA2)
- net MADDR1: now reaches U2.88 (MA1)
- net MADDR10: now reaches U2.92 (MA10)
- net MADDR5: now reaches U2.93 (MA5)
- net MADDR9: now reaches U2.94 (MA9)
- net MADDR7: now reaches U2.95 (MA7)
- net MADDR12: now reaches U2.96 (MA12)
- net MADDR3: now reaches U2.97 (MA3)
- net DDR_BA1: now reaches U2.99 (MBA1)

Commit message: updated
Parts:
- C8: footprint (none) -> Capacitor_SMD:C_0402_1005Metric; LCSC (none) -> C15684
Connections:
- net DDR_IO_1V8_MT7688 renamed DDR_IO_1V8_MT7628
Changed lines of the file:
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@@
+	)
+	(symbol
+		(lib_id "power:+1V8")
+		(at 73.66 88.9 0)
+		(unit 1)
+		(exclude_from_sim no)
+		(in_bom yes)
+		(on_board yes)
+		(dnp no)
+		(fields_autoplaced yes)
+		(property "Reference" "#PWR042"
+			(at 73.66 92.71 0)
+			(effects
+				(font
+					(size 1.27 1.27)
+				)
+				(hide yes)
+			)
+		)
+		(property "Value" "DDR_IO_1V8_MT7628"
+			(at 73.66 83.82 0)
+			(effects
+				(font
+					(size 1.27 1.27)
+				)
+			)
+		)
+		(property "Footprint" ""
+			(at 73.66 88.9 0)
+			(effects
+				(font
+					(size 1.27 1.27)
+				)
+				(hide yes)
+			)
+		)
+		(property "Datasheet" ""
+			(at 73.66 88.9 0)
+			(effects
+				(font
+					(size 1.27 1.27)
+				)
+				(hide yes)
+			)
+		)
+		(property "Description" "Power symbol creates a global label with name \"+1V8\""
+			(at 73.66 88.9 0)
+			(effects
+				(font
+					(size 1.27 1.27)
+				)
+				(hide yes)
+			)
+		)
+		(pin "1"
+		)
+		(instances
+			(project ""
+				(path "/144686d4-2b77-460c-9924-cc86faff7e9d/d136ccdd-d369-41a7-95db-a3b0f1b1dbbd"
+					(reference "#PWR042")
+					(unit 1)
+				)
+			)
+		)
 	)
 	(symbol
@@
 	)
 	(symbol
-		(lib_id "MT7688AN_Power-altium-import:3.3VD_CIRCLE")
-		(at 73.66 88.9 180)
-		(unit 1)
-		(exclude_from_sim no)
-		(in_bom yes)
-		(on_board yes)
-		(dnp no)
-		(property "Reference" "#PWR016"
-			(at 73.66 88.9 0)
-			(effects
-				(font
-					(size 1.27 1.27)
-				)
-				(hide yes)
-			)
-		)
-		(property "Value" "DDR_IO_1V8_MT7688"
-			(at 73.66 85.09 0)
-			(effects
-				(font
-					(size 1.27 1.27)
-				)
-			)
-		)
-		(property "Footprint" ""
-			(at 73.66 88.9 0)
-			(effects
-				(font
-					(size 1.27 1.27)
-				)
-			)
-		)
-		(property "Datasheet" ""
-			(at 73.66 88.9 0)
-			(effects
-				(font
-					(size 1.27 1.27)
-				)
-			)
-		)
-		(property "Description" ""
-			(at 73.66 88.9 0)
-			(effects
-				(font
-					(size 1.27 1.27)
-				)
-			)
-		)
-		(pin ""
-		)
-		(instances
-			(project "mt7628v1"
-				(path "/144686d4-2b77-460c-9924-cc86faff7e9d/d136ccdd-d369-41a7-95db-a3b0f1b1dbbd"
-					(reference "#PWR016")
-					(unit 1)
-				)
-			)
-		)
-	)
-	(symbol
 		(lib_id "mt7628_222:MT7628_*")
 		(at 95.25 72.39 0)
@@
 			)
 		)
-		(property "Footprint" ""
+		(property "Footprint" "Capacitor_SMD:C_0402_1005Metric"
 			(at 73.3552 105.41 0)
 			(effects
@@
 			(at 72.39 101.6 0)
 			(effects
+				(font
+					(size 1.27 1.27)
+				)
+				(hide yes)
+			)
+		)
+		(property "LCSC" "C15684"
+			(at 72.39 101.6 0)
+			(effects

Commit message: f_ver
Parts:
- added C10, C11: 1uf/6.3v, Capacitor_SMD:C_0402_1005Metric, symbol Device:C
- added C12, C13: 1.5nf/50V, Capacitor_SMD:C_0402_1005Metric, symbol Device:C
- added C14, C15, C16, C37, C38, C39, C40: 100nf/16v, Capacitor_SMD:C_0402_1005Metric, symbol DDR2_CFG-altium-import:root_1_Cap_Miscellaneous Devices.SchLib
- added C9: 2.2uF/6.3V, Capacitor_SMD:C_0603_1608Metric, symbol MT7688AN_Power-altium-import:root_3_Cap2_Miscellaneous Devices.SchLib
- U2: footprint MT7628:MT7628_footprint -> Library:MT7628_footprint
Connections:
- net DDR_IO_1V8_MT7628: now also C10.1, C11.1, C12.1, C13.1, C14.2, C15.2, C16.2, C37.2, C38.2, C39.2, C40.2, C9.1
- net GND: now also C10.2, C11.2, C12.2, C13.2, C14.1, C15.1, C16.1, C37.1, C38.1, C39.1, C40.1, C9.2

Commit message: final_all_router by asif
Parts:
- U2: value ~ -> MT7628NN; LCSC (none) -> C2762437
Connections:
- net MADDR13: no longer names the net of U2.83 (MA13)
- no-connect marks 0 -> 1
Changed lines of the file:
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@@
 		(color 0 0 0 0)
 	)
+	(no_connect
+		(at 115.57 78.74)
+	)
 	(wire
 		(pts
@@
 		)
 	)
-	(global_label "MADDR13"
-		(shape input)
-		(at 115.57 78.74 0)
-		(fields_autoplaced yes)
-		(effects
-			(font
-				(size 0.508 0.508)
-			)
-			(justify left)
-		)
-		(property "Intersheetrefs" "${INTERSHEET_REFS}"
-			(at 120.2717 78.74 0)
-			(effects
-				(font
-					(size 1.27 1.27)
-				)
-				(justify left)
-				(hide yes)
-			)
-		)
-	)
 	(global_label "MDATA2"
 		(shape input)
@@
 		(on_board yes)
 		(dnp no)
-		(fields_autoplaced yes)
 		(property "Reference" "#PWR042"
 			(at 73.66 92.71 0)
@@
 		)
 		(property "Value" "DDR_IO_1V8_MT7628"
-			(at 73.66 83.82 0)
+			(at 72.39 84.836 0)
 			(effects
 				(font
@@
 			)
 		)
-		(property "Value" "~"
-			(at 95.25 59.69 0)
+		(property "Value" "MT7628NN"
+			(at 95.504 57.658 0)
 			(effects
 				(font
@@
 			(at 95.25 72.39 0)
 			(effects
+				(font
+					(size 1.27 1.27)
+				)
+				(hide yes)
+			)
+		)
+		(property "LCSC" "C2762437"
+			(at 95.25 72.39 0)
+			(effects
