File: dip.kicad_sch (KiCad schematic)
At the start: 0 parts

Commit message: init_sch
Parts:
- added U4: MT7688_DIP, MT7688_DIP, symbol MT7688AN_DIP_-altium-import:root_0_MT7688_DIP_MT7688_PCBProject.SCHLIB
Connections:
- new net 3.3VD: U4.2 (3.3V_IN)
- new net 5VD: U4.25 (5V_USB)
- new net EPH_LED0_N: U4.34 (EPH_LED0_N)
- new net EPH_LED1_N: U4.32 (EPH_LED1_N)
- new net GND: U4.24 (GND), U4.26 (GND)
- new net GPIO_0: U4.7 (GPIO0)
- new net I2C_SCLK: U4.10 (I2C_SCLK)
- new net I2C_SD: U4.9 (I2C_SD)
- new net I2S_CLK: U4.6 (I2S_CLK)
- new net I2S_DI: U4.8 (I2S_SDI)
- new net I2S_DO: U4.5 (I2S_SDO)
- new net I2S_WS: U4.4 (I2S_WS)
- new net PERST_N: U4.28 (PERST_N)
- new net PWM_CH0: U4.44 (PWM_CH0)
- new net PWM_CH1: U4.43 (PWM_CH1)
- new net REF_CLK0: U4.31 (REF_CLKO)
- new net RXIN0: U4.17 (ETHP0_RN)
- new net RXIN1: U4.23 (ETHP1_RN)
- new net RXIP0: U4.16 (ETHP0_RP)
- new net RXIP1: U4.22 (ETHP1_RP)
- new net SD_CD: U4.38 (SD_CD)
- new net SD_CLK: U4.36 (SD_CLK)
- new net SD_CMD: U4.42 (SD_CMD)
- new net SD_D0: U4.35 (SD_D0)
- new net SD_D1: U4.37 (SD_D1)
- new net SD_D2: U4.41 (SD_D2)
- new net SD_D3: U4.40 (SD_D3)
- new net SD_WP: U4.39 (SD_WP)
- new net SPI_CLK: U4.12 (SPI_CLK)
- new net SPI_CS0: U4.14 (SPI_CS0)
- new net SPI_CS1: U4.11 (SPI_CS1)
- new net SPI_MISO: U4.13 (SPI_MISO)
- new net SPI_MOSI: U4.15 (SPI_MOSI)
- new net TXON0: U4.19 (ETHP0_TN)
- new net TXON1: U4.21 (ETHP1_TN)
- new net TXOP0: U4.18 (ETHP0_TP)
- new net TXOP1: U4.20 (ETHP1_TP)
- new net UART_RXD0: U4.3 (UART_RXD0)
- new net UART_RXD1: U4.29 (UART_RXD1)
- new net UART_RXD2: U4.48 (UART_RXD2)
- new net UART_TXD0: U4.1 (UART_TXD0)
- new net UART_TXD1: U4.27 (UART_TXD1)
- new net UART_TXD2: U4.46 (UART_TXD2)
- new net USB_D+: U4.45 (USB_DP)
- new net USB_D-: U4.47 (USB_DM)
- new net WIFI_RESET: U4.30 (WIFI_RESET)
- new net WLED_N: U4.33 (WLED_N)

Commit message: updated
Parts:
- U4: LCSC (none) -> NC
Changed lines of the file:
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@@
+			)
+		)
+		(property "LCSC" "NC"
+			(at 107.95 50.8 0)
+			(effects
+				(font
+					(size 1.27 1.27)
+				)
+				(hide yes)
 			)
 		)
@@
 			(at 107.95 106.68 0)
 			(effects
+				(font
+					(size 1.27 1.27)
+				)
+				(hide yes)
+			)
+		)
+		(property "LCSC" "NC"
+			(at 107.95 106.68 0)
+			(effects

Commit message: final_all_router by asif
Parts:
- removed U4: MT7688_DIP, MT7688_DIP, symbol MT7688AN_DIP_-altium-import:root_0_MT7688_DIP_MT7688_PCBProject.SCHLIB
