File: power.kicad_sch (KiCad schematic)
At the start: 19 parts

Commit message: updated aux
Parts:
- U2: footprint (none) -> MT7628:MT7628_footprint
Changed lines of the file:
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@@
 			)
 		)
-		(property "Footprint" ""
+		(property "Footprint" "MT7628:MT7628_footprint"
 			(at 149.86 81.28 0)
 			(effects

Commit message: updated
Parts:
- C25: renamed from C5; footprint 0402_C -> Capacitor_SMD:C_0402_1005Metric; LCSC (none) -> C1525
- C26: renamed from C6; footprint 0402_C -> Capacitor_SMD:C_0402_1005Metric; LCSC (none) -> C1525
- C27: renamed from C9; footprint 0603_C -> Capacitor_SMD:C_0603_1608Metric; LCSC (none) -> C71000
- C28: renamed from C12; footprint 0603_C -> Capacitor_SMD:C_0603_1608Metric; LCSC (none) -> C1691
- C29: renamed from C14; footprint 0402_C -> Capacitor_SMD:C_0402_1005Metric; LCSC (none) -> C1525
- C30: renamed from C10; footprint 0402_C -> Capacitor_SMD:C_0402_1005Metric; LCSC (none) -> C15684
- C31: renamed from C11; footprint 0603_C -> Capacitor_SMD:C_0603_1608Metric; LCSC (none) -> C71000
- C32: renamed from C13; footprint 0603_C -> Capacitor_SMD:C_0603_1608Metric; LCSC (none) -> C8032
- C33: footprint 0603_C -> Capacitor_SMD:C_0603_1608Metric; LCSC (none) -> C8032
- C34, C35, C36, C37, C38, C39: footprint 0402_C -> Capacitor_SMD:C_0402_1005Metric; LCSC (none) -> C1525
- C72: renamed from C7; footprint 0402_C -> Capacitor_SMD:C_0402_1005Metric; LCSC (none) -> C1548
- C73: renamed from C8; footprint 0402_C -> Capacitor_SMD:C_0402_1005Metric; LCSC (none) -> C1548
- L1: footprint L2520_TDK -> Inductor_SMD:L_TDK_VLS6045EX_VLS6045AF; LCSC (none) -> NC

Commit message: f_ver
Parts:
- removed C37, C38, C39: 100nf/16v, Capacitor_SMD:C_0402_1005Metric, symbol MT7688AN_Power-altium-import:root_1_Cap_Miscellaneous Devices.SchLib
- L1: footprint Inductor_SMD:L_TDK_VLS6045EX_VLS6045AF -> Library:IND_VLS252012ET-100M
- U2: footprint MT7628:MT7628_footprint -> Library:MT7628_footprint
Connections:
- net SOC_1.2VD_MT7688 is gone; now on net SOC_1.2VD_MT7628: C28.1, C29.2, C33.1, C34.2, C35.2, C36.2, L1.2, U2.122 (VOUT_FB)

Commit message: final_all_router by asif
Parts:
- added C74, C89, C90, C91, C92, C93: 22uf/25v, Capacitor_SMD:C_0603_1608Metric, symbol Device:C
- added C75: 10uf/6.3v, Capacitor_SMD:C_0603_1608Metric, symbol Device:C
- added C76: 100nf/16v, Capacitor_SMD:C_0402_1005Metric, symbol MT7688AN_Power-altium-import:root_1_Cap_Miscellaneous Devices.SchLib
- added C78: 470uf/25v, easyeda2kicad:CAP-TH_BD8.0-P3.50-D0.6-FD, symbol Device:C
- added C84: 10uf/25v, Capacitor_SMD:C_0603_1608Metric, symbol Device:C
- added C85: 100nf/16v, Capacitor_SMD:C_0402_1005Metric, symbol Device:C
- added C86, C87, C94: NC, Capacitor_SMD:C_0402_1005Metric, symbol Device:C
- added C88: 1uf/25v, Capacitor_SMD:C_0402_1005Metric, symbol Device:C
- added D3: LED, Diode_SMD:D_0603_1608Metric, symbol Device:LED
- added J1: Barrel_Jack_Switch, easyeda2kicad:DC-IN-TH_DC-005C-20A, symbol Connector:Barrel_Jack_Switch
- added L11: 6.8uh, easyeda2kicad:IND-SMD_L4.5-W4.0_GCD43-XX, symbol Device:L
- added R39: 510/0402, Resistor_SMD:R_0402_1005Metric, symbol Device:R
- added R46: 100K/0402, Resistor_SMD:R_0402_1005Metric, symbol Device:R
- added R47: 1k/1%, Resistor_SMD:R_0402_1005Metric, symbol DDR2_CFG-altium-import:root_1_Res1_Miscellaneous Devices.SchLib
- added R48: 6.2K/0603, Capacitor_SMD:C_0603_1608Metric, symbol Device:R
- added R49: 2K/0402, Capacitor_SMD:C_0402_1005Metric, symbol Device:R
- added U4: ams1117-5v, easyeda2kicad:SOT-223_L6.5-W3.5-P2.30-LS7.0-BR, symbol ams117:ams117-5v
- added U7: MP1470, Package_TO_SOT_SMD:TSOT-23-6, symbol Regulator_Switching:MP1470
- L1: value 2.2 uH/VLS252012T-2R2M1R3 -> 2.2 uH/VLS252012ET-2R2M; footprint Library:IND_VLS252012ET-100M -> easyeda2kicad:IND-SMD_L2.5-W2.0_VLS2520X; LCSC NC -> C107346
- U2: value ~ -> MT7628NN; LCSC (none) -> C2762437
Connections:
- net 3.3VD: now also C89.1, C90.1, C91.1, C92.1, C93.1, C94.2, L11.2, R39.1, R48.1
- net GND: now also C74.2, C75.2, C76.1, C78.2, C84.2, C85.2, C86.2, C87.2, C89.2, C90.2, C91.2, C92.2, C93.2, D3.1 (K), J1.2, J1.3, R49.2, U4.1 (GND), U7.1 (GND)
- new net: D3.2 (A), R39.2
- new net: C86.1, C87.1, R46.1, U7.5 (EN)
- new net: C94.1, R47.1, R48.2, R49.1
- new net: C88.2, L11.1, U7.2 (SW)
- new net: R47.2, U7.4 (FB)
- new net: C88.1, U7.6 (BST)
- new net +12V: C74.1, C78.1, C84.1, C85.1, J1.1, R46.2, U4.3 (VIN), U7.3 (IN)
- new net +5V: C75.1, C76.2, U4.2 (VOUT), U4.4 (VOUT)
