File: reset.kicad_sch (KiCad schematic)
At the start: 0 parts

Commit message: init_sch
Parts:
- added C77: 4.7uf/6.3v, 0603_C, symbol MT7688AN_Reset-altium-import:root_3_Cap2_Miscellaneous Devices.SchLib
- added D1, D2: LED0, 0603_LED_S1, symbol MT7688AN_Reset-altium-import:root_0_mirrored_LED0_Miscellaneous Devices.SchLib
- added R34: 20K/1%, 0402_R, symbol MT7688AN_Reset-altium-import:root_1_Res1_Miscellaneous Devices.SchLib
- added R35: 22, 0402_R, symbol MT7688AN_Reset-altium-import:root_2_Res1_Miscellaneous Devices.SchLib
- added R36, R37: 330, 0402_R, symbol MT7688AN_Reset-altium-import:root_2_Res1_Miscellaneous Devices.SchLib
Connections:
- new net: D2.1 (A), R37.2
- new net: D1.1 (A), R36.2
- new net: C77.1, R34.1, R35.2
- new net 3.3VD: R34.2, R36.1, R37.1
- new net CPURST_N: R35.1
- new net GND: C77.2, D2.2 (K)
- new net WLED_N: D1.2 (K)

Commit message: updated
Parts:
- C77: footprint 0603_C -> Capacitor_SMD:C_0603_1608Metric; LCSC (none) -> C8032
Changed lines of the file:
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@@
 			)
 		)
-		(property "Footprint" "0603_C"
+		(property "Footprint" "Capacitor_SMD:C_0603_1608Metric"
 			(at 100.33 85.09 0)
 			(effects
@@
 				(hide yes)
 			)
+		)
+		(property "LCSC" "C8032"
+			(at 100.33 85.09 0)
+			(effects
+				(font
+					(size 1.27 1.27)
+				)
+				(hide yes)
+			)

Commit message: f_ver
Parts:
- D1, D2: footprint 0603_LED_S1 -> LED_SMD:LED_0603_1608Metric; LCSC (none) -> C9900005774
- R34: footprint 0402_R -> Resistor_SMD:R_0402_1005Metric; LCSC (none) -> C25545
- R35: footprint 0402_R -> Resistor_SMD:R_0402_1005Metric; LCSC (none) -> C25092
- R36, R37: footprint 0402_R -> Resistor_SMD:R_0402_1005Metric; LCSC (none) -> C25104
Changed lines of the file:
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@@
 			)
 		)
-		(property "Footprint" "0402_R"
+		(property "Footprint" "Resistor_SMD:R_0402_1005Metric"
 			(at 158.75 128.27 0)
 			(effects
@@
 				)
 				(justify left bottom)
+				(hide yes)
+			)
+		)
+		(property "LCSC" "C25104"
+			(at 158.75 128.27 0)
+			(effects
+				(font
+					(size 1.27 1.27)
+				)
 				(hide yes)
 			)
@@
 			)
 		)
-		(property "Footprint" "0402_R"
+		(property "Footprint" "Resistor_SMD:R_0402_1005Metric"
 			(at 158.75 115.57 0)
 			(effects
@@
 				)
 				(justify left bottom)
+				(hide yes)
+			)
+		)
+		(property "LCSC" "C25104"
+			(at 158.75 115.57 0)
+			(effects
+				(font
+					(size 1.27 1.27)
+				)
 				(hide yes)
 			)
@@
 			)
 		)
-		(property "Footprint" "0402_R"
+		(property "Footprint" "Resistor_SMD:R_0402_1005Metric"
 			(at 95.25 69.85 0)
 			(effects
@@
 				)
 				(justify left bottom)
+				(hide yes)
+			)
+		)
+		(property "LCSC" "C25545"
+			(at 95.25 69.85 0)
+			(effects
+				(font
+					(size 1.27 1.27)
+				)
 				(hide yes)
 			)
@@
 			)
 		)
-		(property "Footprint" "0402_R"
+		(property "Footprint" "Resistor_SMD:R_0402_1005Metric"
 			(at 113.03 80.01 0)
 			(effects
@@
 				)
 				(justify left bottom)
+				(hide yes)
+			)
+		)
+		(property "LCSC" "C25092"
+			(at 113.03 80.01 0)
+			(effects
+				(font
+					(size 1.27 1.27)
+				)
 				(hide yes)
 			)
@@
 			)
 		)
-		(property "Footprint" "0603_LED_S1"
+		(property "Footprint" "LED_SMD:LED_0603_1608Metric"
 			(at 125.73 110.49 0)
 			(effects
@@
 				)
 				(justify left bottom)
+				(hide yes)
+			)
+		)
+		(property "LCSC" "C9900005774"
+			(at 125.73 110.49 0)
+			(effects
+				(font
+					(size 1.27 1.27)
+				)
 				(hide yes)
 			)
@@
 			)
 		)
-		(property "Footprint" "0603_LED_S1"
+		(property "Footprint" "LED_SMD:LED_0603_1608Metric"
 			(at 125.73 123.19 0)
 			(effects
@@
 				(hide yes)
 			)
+		)
+		(property "LCSC" "C9900005774"
+			(at 125.73 123.19 0)
+			(effects
+				(font
+					(size 1.27 1.27)
+				)
+				(hide yes)
+			)

Commit message: final_all_router by asif
Parts:
- D1, D2: LCSC C9900005774 -> C2286
Changed lines of the file:
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@@
 			)
 		)
-		(property "LCSC" "C9900005774"
+		(property "LCSC" "C2286"
 			(at 125.73 110.49 0)
 			(effects
@@
 			)
 		)
-		(property "LCSC" "C9900005774"
-			(at 125.73 123.19 0)
-			(effects
+		(property "LCSC" "C2286"
+			(at 125.73 123.19 0)
+			(effects
